File: FishIoT/FishIoT.kicad_sch (KiCad schematic)
At the start: 122 parts, among them IC1 RV-3032-C7_32.768KHZ-2.5PPM-T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, J1 VDD_JUMPER, J10 RM_UART, J11 Current Measurement, J13 UART_DEBUG, J2 0705430001, J3 SF72S006VBDR2500, J4 SHF-105-01-L-D-SM, J5 10119313-302TLF, J6 BM05B-ZESS-TBT, J8 BM05B-ZESS-TBT, J9 Conn_Coaxial, SW1 PTS645SM43SMTR92 LF, SW2 PTS645SM43SMTR92 LF, SW3 PTS645SM43SMTR92 LF, U1 NRF9160-SICA, U10 RM126x, U2 SKY65943-11, U3 TPD3F303DPVR, U4 TPS63000, U5 USBLC6-2P6, U6 CP2102N-Axx-xQFN20, U9 MAX3471

Commit message: v26.0
First draft of schematics and PCB with nRF9151
Parts:
- removed ANT1: P822601, FishIoT_Footprint_library:ANT_P822601, symbol FishIoTSymbol_Library.Library:P822601
- removed BT1: 3002, FishIoT_Footprint_library:BAT_3002, symbol FishIoTSymbol_Library.Library:3002
- removed C1: C, Capacitor_SMD:C_0603_1608Metric, symbol Device:C
- removed C10, C11: 100pF, Capacitor_SMD:C_0603_1608Metric, symbol Device:C
- removed C12, C13, C9: 100nF, Capacitor_SMD:C_0603_1608Metric, symbol Device:C
- removed C14: 4.7uF, Capacitor_SMD:C_0603_1608Metric, symbol Device:C
- removed C19: 47uF, Capacitor_SMD:C_0603_1608Metric, symbol Device:C
- removed C2: 100n, Capacitor_SMD:C_0603_1608Metric, symbol Device:C
- removed H3: MountingHole_Pad, MountingHole:MountingHole_3mm_Pad_Via, symbol Mechanical:MountingHole_Pad
- removed J10: RM_UART, Connector_PinHeader_2.54mm:PinHeader_1x03_P2.54mm_Vertical, symbol Connector:Conn_01x03_Socket
- removed J13: UART_DEBUG, Connector_PinHeader_2.54mm:PinHeader_1x03_P2.54mm_Vertical, symbol Connector:Conn_01x03_Socket
- removed J3: SF72S006VBDR2500, FishIoT_Footprint_library:JAE_SF72S006VBDR2500, symbol FishIoTSymbol_Library.Library:SF72S006VBDR2500
- removed J5: 10119313-302TLF, FishIoT_Footprint_library:AMPHENOL_10119313-302TLF, symbol Connector:USB_B
- removed J6: BM05B-ZESS-TBT, FishIoT_Footprint_library:BM05BZESSTBTLFSN, symbol Connector:Conn_01x05_Socket
- removed J9: Conn_Coaxial, FishIoT_Footprint_library:LINX_CONUFL001-SMD-T, symbol Connector:Conn_Coaxial
- removed L3: L, Inductor_SMD:L_0603_1608Metric, symbol Device:L
- removed L4, L7: 33nH, Inductor_SMD:L_0603_1608Metric, symbol Device:L
- removed L5: 9.1nH, Inductor_SMD:L_0603_1608Metric, symbol Device:L
- removed PPS1, RTC_CO1, VSIM1: TestPoint, TestPoint:TestPoint_Pad_D1.0mm, symbol Connector:TestPoint
- removed R2: 1M0, Resistor_SMD:R_0603_1608Metric, symbol Device:R
- removed R27, R32: 0, Resistor_SMD:R_0603_1608Metric, symbol Device:R
- removed R37: 100, Resistor_SMD:R_0603_1608Metric, symbol Device:R
- removed RTC_EVI1: RTC_EVI, TestPoint:TestPoint_Pad_D1.0mm, symbol Connector:TestPoint
- removed U1: NRF9160-SICA, FishIoT_Footprint_library:XCVR_NRF9160-SICA, symbol FishIoTSymbol_Library.Library:NRF9160-SICA
- removed U10: RM126x, FishIoT_Footprint_library:Laird, RM126X, symbol FishIoTSymbol_Library.Library:RM126x
- removed U2: SKY65943-11, FishIoT_Footprint_library:IC_SKY65943-11, symbol FishIoTSymbol_Library.Library:SKY65943-11
- removed U3: TPD3F303DPVR, FishIoT_Footprint_library:SON50P210X160X65-9N, symbol FishIoTSymbol_Library.Library:TPD3F303DPVR
- added C15: 100nF, Capacitor_SMD:C_0603_1608Metric, symbol Device:C
- added C16: TBD, Capacitor_SMD:C_0603_1608Metric, symbol Device:C
- added C26: 10u, Capacitor_SMD:C_0603_1608Metric, symbol Device:C
- added C5: 100n, Capacitor_SMD:C_0603_1608Metric, symbol Device:C
- added D+1, D-1, GPIO_0.11, GPIO_P.016, LNA_EN1, UART_RX1, UART_TX1: TestPoint, TestPoint:TestPoint_Pad_D1.0mm, symbol Connector:TestPoint
- added J1: USB4105-GF-A-120, Footprints:GCT_USB4105-GF-A-120, symbol USB4105-GF-A-120:USB4105-GF-A-120
- added J3, J6: Conn_Coaxial, Footprints:LINX_CONUFL001-SMD-T, symbol Connector:Conn_Coaxial
- added J5: SF72S006VBDR2500, Footprints:JAE_SF72S006VBDR2500, symbol FishIoTSymbol_Library.Library:SF72S006VBDR2500
- added JP1, JP2: SolderJumper_2_Open, Jumper:SolderJumper-2_P1.3mm_Open_RoundedPad1.0x1.5mm, symbol Jumper:SolderJumper_2_Open
- added R18: 10, Resistor_SMD:R_0603_1608Metric, symbol Device:R
- added R29: 10k, Resistor_SMD:R_0603_1608Metric, symbol Device:R
- added R3: 5.1k, Resistor_SMD:R_0603_1608Metric, symbol Device:R
- added U2: NRF9151-LACA-R7, NRF9151_LACA_R7:XCVR_NRF9151-LACA-R7, symbol NRF9151-LACA-R7:NRF9151-LACA-R7
- added U4: MAX-M10S, RF_GPS:ublox_MAX, symbol RF_GPS:MAX-M10S
- added U5: TPD3F303DPVR, Footprints:SON50P210X160X65-9N, symbol FishIoTSymbol_Library.Library:TPD3F303DPVR
- added U7: SI1040X-T1-GE3, Footprints:SON_0X-T1-GE3_VIS, symbol SON_0X-T1-GE3:SI1040X-T1-GE3
- C1: renamed from C23; value 15p -> 1u
- C17: value 15p -> 10nF
- C2: renamed from C22; value 100n -> 1u
- C3: renamed from C21; value 47u -> 10u
- C6: renamed from C18; value 100n -> 10u
- J4: renamed from J8; footprint FishIoT_Footprint_library:BM05BZESSTBTLFSN -> Footprints:BM05BZESSTBTLFSN
- J7: renamed from J4; footprint FishIoT_Footprint_library:SHF-105-01-X-D-SM -> Footprints:SHF-105-01-X-D-SM
- J8: renamed from J2; footprint FishIoT_Footprint_library:MOLEX_0705430001 -> Footprints:MOLEX_0705430001
- L1: value 1.5nH -> TBD; now left out of the parts list
- L2: value 22nH -> 27nH
- R1: value 0R -> 5.1k
- R16: value R -> 0
- R17: value 120 -> 100k
- R34: renamed from R8; value 240k -> 215k
- renumbered C20 to C10, C30 to C11, C28 to C12, C33 to C13, C32 to C14, C7 to C18, C24 to C19, C25 to C20, C5 to C21, C6 to C22, C8 to C23, C27 to C24, C26 to C25, C16 to C4, C15 to C7, C29 to C8, C31 to C9, D6 to D7, J11 to JP3, J1 to JP4, L6 to L3, R29 to R11, R30 to R12, R36 to R13, R35 to R14, R34 to R15, R24 to R19, R3 to R2, R6 to R25, R25 to R26, R33 to R27, R26 to R28, R31 to R30, R14 to R31, R15 to R32, R7 to R33, R5 to R4, R4 to R5, R9 to R6, R11 to R7, R12 to R8, R13 to R9, U5 to U1, U6 to U3, U9 to U6, U4 to U8
Connections:
- net GPS_RF_ANT is gone; now on an unnamed net: R16.1
- net LTE_RF1 is gone; now on net GND: L1.1
- net TBR_PPS is gone; now on net RTC_CLKOUT: J4.4 (Pin_4)
- net +3V3: now also C26.2, U2.65 (VDD_GPIO), U4.7 (VCC_IO), U4.8 (VCC); no longer C17.1, C6.1
- net Battery_voltage: now also U2.78 (P0.17/AIN4)
- net GND: now also R1.1, C15.1, C16.2, C26.1, C5.1, J1.A1_B12 (GND), J1.B1_A12 (GND__1), J3.2 (Ext), J5.C5 (GND), J5.G1 (SHIELD), J5.G10 (SHIELD), J5.G2 (SHIELD), J5.G3 (SHIELD), J5.G4 (SHIELD), J5.G5 (SHIELD), J5.G6 (SHIELD), J5.G7 (SHIELD), J5.G8 (SHIELD), J5.G9 (SHIELD), J6.2 (Ext), R29.1, R3.2, U2.1 (GND_1), U2.105 (GND_2__6), U2.106 (GND_2__7), U2.107 (GND_2__8), U2.108 (GND_2__9), U2.109 (GND_2__10), U2.110 (GND_2__11), U2.111 (GND_2__12), U2.112 (GND_2__13), U2.113 (GND_2__14), U2.13 (GND_1__2), U2.15 (GND_1__3), U2.20 (GND_1__4), U2.25 (GND_1__5), U2.30 (GND_1__6), U2.34 (GND_1__7), U2.36 (GND_1__8), U2.38 (GND_1__9), U2.39 (GND_1__10), U2.40 (GND_1__11), U2.41 (GND_1__12), U2.43 (GND_1__13), U2.46 (GND_1__14), U2.51 (GND_2), U2.55 (GND_2__1), U2.60 (GND_2__2), U2.66 (GND_2__3), U2.7 (GND_1__1), U2.71 (GND_2__4), U2.76 (GND_2__5), U4.1 (GND), U4.10 (GND), U4.12 (GND), U5.9 (GND), U7.1 (R2); no longer L2.1
- net I2C_SCL: now also U2.63 (P0.06)
- net I2C_SDA: now also U2.62 (P0.05)
- net PPS: now also IC1.4 (EVI), R30.2, JP2.2 (B), U4.4 (TIMEPULSE)
- net RS485_A: now also R13.2; no longer R13.1
- net RS485_B: now also R13.1; no longer R13.2
- net RS485_DE: now also U2.73 (P0.13/AIN0)
- net RS485_DI: now also U2.72 (P0.12)
- net RS485_RE: now also U2.74 (P0.14/AIN1)
- net RS485_RX: now also U2.75 (P0.15/AIN2)
- net SIM_CLK: now also U2.18 (SIM_CLK), U5.7 (CLK_IN)
- net SIM_IO: now also U2.17 (SIM_IO), U5.6 (DATA2_IN)
- net SIM_RST: now also U2.16 (SIM_RST), U5.8 (DATA1_IN)
- net SIM_VCC: now also C15.2, J5.C1 (VCC), U2.19 (SIM_1V8), U5.5 (VCC)
- net SWDCLK: now also U2.3 (SWDCLK)
- net SWDIO: now also U2.4 (SWDIO)
- net UART1_RX: now also U2.58 (P0.02), U4.3 (RXD)
- net UART1_TX: now also U2.59 (P0.03), U4.2 (TXD)
- net nINT_RTC: now also U2.61 (P0.04)
- net nRF91_BUTTON1: now also U2.5 (P0.21/TRACECLK)
- net nRF91_BUTTON2: now also U2.6 (P0.22/TRACEDATA(0))
- net nRF91_LED1: now also U2.48 (P0.29)
- net nRF91_LED2: now also U2.47 (P0.28)
- net nRF91_LED3: now also U2.45 (P0.27)
- net nRF91_LED4: now also U2.44 (P0.26)
- net nRF_UART_RX: now also U2.79 (P0.18/AIN5), UART_RX1.1
- net nRF_UART_TX: now also U2.80 (P0.19/AIN6), UART_TX1.1
- net ~{nRESET}: now also J7.10, R2.2; no longer R1.2, R2.1
- net at R4.1: now also U2.54 (COEX2)
- net D+: now reaches R6.1, U1.1 (I/O1), U1.6 (I/O1)
- net D+: now also D+1.1, J1.A6 (DP1), J1.B6 (DP2)
- net D-: now reaches R10.1, U1.3 (I/O2), U1.4 (I/O2)
- net D-: now also D-1.1, J1.A7 (DN1), J1.B7 (DN2)
- net VUSB_C: now reaches FB2.2, U1.5 (VBUS)
- net VUSB_C: now also J1.A4_B9 (VBUS), J1.B4_A9 (VBUS__1)
- net at R16.2: now also L2.1, C16.1, J6.1 (In)
- net at FB1.2, R5.1: now also C6.1, U2.14 (VDD)
- net at R5.2: now also U2.10 (ENABLE)
- net at C4.2: now also R2.1, U2.9 (~{RESET}); no longer R2.2
- net at L1.2: now also U4.11 (RF_IN); no longer L2.2
- net at R17.2: now also U4.14 (VCC_RF), U7.4 (S2); no longer IC1.1 (VBACKUP)
- net at R17.1: now also U7.6 (R1,_C1)
- net RTC_CLOCKOUT renamed RTC_CLKOUT
- net RTC_CLKOUT: now also JP1.2 (B)
- net VBUS renamed VUSB
- new net: GPIO_0.11.1, U2.70 (P0.11)
- new net: JP2.1 (A), U2.57 (P0.01)
- new net: LNA_EN1.1, U4.13 (LNA_EN), U7.5 (ON/OFF)
- new net: GPIO_P.016.1, U2.77 (P0.16/AIN3)
- new net: J3.1 (In), U2.35 (ANT)
- new net: JP1.1 (A), U2.64 (P0.07)
- new net: J5.C2 (RST), U5.1 (DATA1_OUT)
- new net: J5.C3 (CLK), U5.2 (CLK_OUT)
- new net: J5.C7 (I/O), U5.3 (DATA2_OUT)
- new net: J1.A5 (CC1), R1.2
- new net: J1.B5 (CC2), R3.1
- new net: C5.2, J1.SH4 (SHELL_GND__3)
- new net: IC1.1 (VBACKUP), R29.2
- new net: C17.1, L2.2, R18.1
- new net: R18.2, U7.2 (D2), U7.3 (D2)
- new net GPS_EXTINT: U2.56 (P0.00), U4.5 (EXTINT)
- no-connect marks 23 -> 38
Other:
- note added: "GNSS"
- note added: "J-LINK"
- note added: "Optional active antenna power"
- note added: "Optional read"
- note added: "RS485"
- note added: "USB-C to UART"
- note added: "VDD selector and Buck-Boost converter"
- note added: "Warning: interal pull-up to 2.2V"
- note added: "impedance matching"
- note added: "nRF9151"
- note removed: "Auxillary UART"
- note removed: "DEBUG"
- note removed: "GPS"
- note removed: "RM126x LoRa Controller"
- note removed: "RS485 Connector"
- note removed: "RS485 controller"
- note removed: "USB and UART-to-USB converter"
- note removed: "VDD selector and Buck converter"
- note removed: "nRF9160"
- company: NTNU Cybernetics Dept Master's Project -> NTNU
- title: IoF (Internet of Fish) nRF9160 board -> IoF (Internet of Fish) nRF9151 board
- moved on the sheet: C1, C10, C11, C12, C13, C14, C18, C19, C2, C20, C21, C22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

Commit message: Added LoRa module
Parts:
- removed GPIO_0.11: TestPoint, TestPoint:TestPoint_Pad_D1.0mm, symbol Connector:TestPoint
- added GPIO_P.024, GPIO_P.025: TestPoint, TestPoint:TestPoint_Pad_D1.0mm, symbol Connector:TestPoint
- added R37: 10k, Resistor_SMD:R_0603_1608Metric, symbol Device:R
- added U9: RM126x, FishIoT_Footprint_library:Laird, RM126X, symbol FishIoTSymbol_Library.Library:RM126x
Connections:
- net +3V3: now also R37.2, U9.10 (VDD_IO), U9.3 (VDD_RADIO), U9.36 (VDD_SX1262), U9.8 (VMCU)
- net Battery_voltage: now also U2.50 (P0.31); no longer U2.78 (P0.17/AIN4)
- net GND: now also U9.1 (GND), U9.11 (GND), U9.2 (GND), U9.21 (GND), U9.24 (GND), U9.25 (GND), U9.26 (GND), U9.28 (GND), U9.29 (GND), U9.30 (GND), U9.31 (GND), U9.35 (GND), U9.4 (GND), U9.40 (GND), U9.41 (GND), U9.42 (GND), U9.43 (GND), U9.44 (GND), U9.45 (GND), U9.46 (GND), U9.47 (GND), U9.7 (GND), U9.9 (GND)
- net RS485_DE: now also U2.68 (P0.09); no longer U2.73 (P0.13/AIN0)
- net RS485_DI: now also U2.67 (P0.08); no longer U2.72 (P0.12)
- net RS485_RE: now also U2.69 (P0.10); no longer U2.74 (P0.14/AIN1)
- net RS485_RX: now also U2.70 (P0.11); no longer U2.75 (P0.15/AIN2)
- net at U2.11 (P0.24/TRACEDATA(2)): now also GPIO_P.024.1
- net at U2.12 (P0.25/TRACEDATA(3)): now also GPIO_P.025.1
- new net BOOT: R37.1, U9.19 (PC06)
- new net RM_CTS: U2.72 (P0.12), U9.32 (PB04)
- new net RM_RESETn: U2.78 (P0.17/AIN4), U9.20 (RESETn)
- new net RM_RTS: U2.74 (P0.14/AIN1), U9.34 (PB02)
- new net RM_RX: U2.73 (P0.13/AIN0), U9.33 (PB03)
- new net RM_TX: U2.75 (P0.15/AIN2), U9.18 (PC07)
- no-connect marks 38 -> 46
Other:
- note added: "COEX2 is high when LTE, GPS or NR+ is active"
- note added: "RM126x LoRa Controller"
- note removed: "When COEX2 is high, LTE or GPS RF is active, when it is low LTE or GPS RF is inactive"
- moved on the sheet: C1, C10, C11, C12, C13, C14, C15, C16, C17, C18, C19, C2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

Commit message: Schematics cleanup
Connections:
- net UART1_RX renamed GNSS_UART_RX
- net UART1_TX renamed GNSS_UART_TX
- net nRF_UART_RX renamed USBC_UART_RX
- net nRF_UART_TX renamed USBC_UART_TX
- no-connect marks 46 -> 47
Other:
- note added: "VDD selector and Buck-Boost regulator"
- note removed: "COEX2 is high when LTE, GPS or NR+ is active"
- note removed: "VDD selector and Buck-Boost converter"
- moved on the sheet: JP2
Changed lines of the file:
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@@
 	(title_block
 		(title "IoF (Internet of Fish) nRF9151 board")
-		(date "2026-02-01")
+		(date "2026-05-23")
 		(rev "version 26.0")
 		(company "NTNU")
@@
 		)
 	)
-	(text "VDD selector and Buck-Boost converter"
+	(text "VDD selector and Buck-Boost regulator"
 		(exclude_from_sim no)
 		(at 409.956 20.066 0)
@@
 		)
 	)
-	(text "COEX2 is high when LTE, \nGPS or NR+ is active\n\n\n"
-		(exclude_from_sim no)
-		(at 74.93 111.506 0)
-		(effects
-			(font
-				(size 1.27 1.27)
-			)
-			(justify right bottom)
-		)
-	)
 	(text "USB-C to UART\n"
 		(exclude_from_sim no)
@@
 	)
 	(no_connect
+		(at 236.22 67.31)
+	)
+	(no_connect
 		(at 144.78 54.61)
 	)
@@
 	(wire
 		(pts
-			(xy 64.77 120.65) (xy 69.85 120.65)
+			(xy 64.77 120.65) (xy 66.04 120.65)
 		)
 		(stroke
@@
 	(wire
 		(pts
-			(xy 77.47 120.65) (xy 93.98 120.65)
+			(xy 73.66 120.65) (xy 93.98 120.65)
 		)
 		(stroke
@@
 		)
 	)
-	(label "nRF_UART_RX"
+	(label "USBC_UART_RX"
 		(at 152.4 100.33 0)
 		(effects
@@
 		)
 	)
-	(label "UART1_RX"
+	(label "GNSS_UART_RX"
 		(at 281.94 133.35 180)
 		(effects
@@
 		)
 	)
-	(label "UART1_TX"
+	(label "GNSS_UART_TX"
 		(at 281.94 135.89 180)
 		(effects
@@
 		)
 	)
-	(label "nRF_UART_RX"
+	(label "USBC_UART_RX"
 		(at 201.93 337.82 0)
 		(effects
@@
 		)
 	)
-	(label "nRF_UART_TX"
+	(label "USBC_UART_TX"
 		(at 201.93 340.36 0)
 		(effects
@@
 		)
 	)
-	(label "UART1_TX"
+	(label "GNSS_UART_TX"
 		(at 86.36 125.73 180)
 		(effects
@@
 		)
 	)
-	(label "nRF_UART_TX"
+	(label "USBC_UART_TX"
 		(at 152.4 102.87 0)
 		(effects
@@
 		)
 	)
-	(label "UART1_RX"
+	(label "GNSS_UART_RX"
 		(at 86.36 123.19 180)
 		(effects
@@
 	(symbol
 		(lib_id "Jumper:SolderJumper_2_Open")
-		(at 73.66 120.65 180)
+		(at 69.85 120.65 180)
 		(unit 1)
 		(exclude_from_sim no)
@@
 		(dnp no)
 		(property "Reference" "JP2"
-			(at 73.66 123.19 0)
+			(at 69.85 123.19 0)
 			(effects
 				(font
@@
 		)
 		(property "Value" "SolderJumper_2_Open"
-			(at 73.66 122.428 0)
+			(at 69.85 122.428 0)
 			(effects
 				(font
@@
 		)
 		(property "Footprint" "Jumper:SolderJumper-2_P1.3mm_Open_RoundedPad1.0x1.5mm"
-			(at 73.66 120.65 0)
+			(at 69.85 120.65 0)
 			(effects
 				(font
@@
 		)
 		(property "Datasheet" "~"
-			(at 73.66 120.65 0)
+			(at 69.85 120.65 0)
 			(effects
 				(font
@@
 		)
 		(property "Description" "Solder Jumper, 2-pole, open"
-			(at 73.66 120.65 0)
+			(at 69.85 120.65 0)
 			(effects
 				(font
@@
 		(dnp no)
 		(property "Reference" "C4"
-			(at 62.23 55.88 90)
+			(at 64.262 56.642 90)
 			(effects
 				(font
@@
 		)
 		(property "Value" "100n"
-			(at 67.31 54.61 90)
+			(at 67.31 54.356 90)
 			(effects
 				(font
@@
 		(fields_autoplaced yes)
 		(property "Reference" "U3"
-			(at 186.3441 388.62 0)
+			(at 186.2933 388.62 0)
 			(effects
 				(font
@@
 		)
 		(property "Value" "CP2102N-Axx-xQFN20"
-			(at 186.3441 391.16 0)
+			(at 186.2933 391.16 0)
 			(effects
 				(font
@@
 		(dnp no)
 		(property "Reference" "R2"
-			(at 67.31 62.23 90)
+			(at 65.278 67.056 90)
 			(effects
 				(font
@@
 		)
 		(property "Value" "1k"
-			(at 67.31 67.31 90)
+			(at 68.834 67.056 90)
 			(effects
 				(font

Commit message: fixed battery measurement, DEC0 capacitor and I2C for GNSS
Parts:
- added C27: 4.7uF, Capacitor_SMD:C_0603_1608Metric, symbol Device:C
- added GPIO_P0.30, GPIO_P0.31: TestPoint, TestPoint:TestPoint_Pad_D1.0mm, symbol Connector:TestPoint
Connections:
- net Battery_voltage: now also U2.2 (P0.20/AIN7); no longer U2.50 (P0.31)
- net GND: now also C27.2
- net GNSS_SDA: now reaches U4.16 (SDA)
- net GNSS_SDA: now also U2.58 (P0.02)
- net GNSS_SCL: now reaches U4.17 (SCL)
- net GNSS_SCL: now also U2.59 (P0.03)
- net at U2.24 (DEC0): now also C27.1
- net at U2.49 (P0.30): now also GPIO_P0.30.1
- net GNSS_UART_RX: no longer names the net of U4.3 (RXD)
- net GNSS_UART_RX: no longer U2.58 (P0.02)
- net GNSS_UART_TX: no longer names the net of U4.2 (TXD)
- net GNSS_UART_TX: no longer U2.59 (P0.03)
- new net: GPIO_P0.31.1, U2.50 (P0.31)
- no-connect marks 47 -> 46
Other:
- moved on the sheet: C10, C7, Vgpio1
